File: LC.kicad_sch (KiCad schematic)
At the start: 86 parts, among them J1 INPUT+, J10 DISPLAY, J11 ENTER_BUTTON, J12 UP_BUTTON, J2 INPUT-, J3 Barrel_Jack, J4 EXT_CLK, J5 CLKSRC, J6 SIGSRC, J7 EXT_SIG, J8 UNUSED, J9 PROG, Q1 BC817, Q2 BC817, SW1 RESET_BTN, U1 Omron_G2V, U10 74HC590PW,118, U11 74HCS251, U12 AVR32DB28x-xSO, U2 L7805, U3 74AHC1G04, U4 Omron_G2E, U5 74AHC1G14, U6 74AHC1G04, U7 LT1719CS6, U8 74AUC1G74, U9 74AUC2G125, Y1 10MHz

Commit message: Updated schematic for 5V devices in TIC, PCB is in todo
Parts:
- removed U9: 74AUC2G125, Package_SO:VSSOP-8_2.4x2.1mm_P0.5mm, symbol 74xGxx:74AUC2G125
- added U10, U9: 74LVC1G125SE-7, Package_TO_SOT_SMD:SOT-353_SC-70-5, symbol 74xGxx:74AUC1G125
- C19: value 470p -> 680p
- R13: value 200R -> 150R
- U8: value 74AUC1G74 -> 74LVC2G74DP,125; footprint Package_SO:VSSOP-8_2.3x2mm_P0.5mm -> Package_SO:TSSOP-8_3x3mm_P0.65mm
- renumbered U10 to U11, U11 to U12, U12 to U13
Connections:
- net +5V: now also U10.5 (VCC), U9.5 (VCC)
- net GND: now also U10.3 (GND), U9.1, U9.3 (GND)
- net SIG_RED: now also U10.2
- net at R13.2: now also U10.4
- net at U8.5 (Q): now also U9.2
- new net: U10.1, U9.4
Changed lines of the file:
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@@
   (symbol (lib_id "74xx_IEEE:74251") (at 262.255 142.875 0) (unit 1)
     (in_bom yes) (on_board yes)
-    (property "Reference" "U11" (id 0) (at 262.255 140.97 0))
+    (property "Reference" "U12" (id 0) (at 262.255 140.97 0))
     (property "Value" "74HCS251" (id 1) (at 268.605 162.56 0))
     (property "Footprint" "Package_SO:SOIC-16_4.55x10.3mm_P1.27mm" (id 2) (at 262.255 142.875 0)
@@
     (pin "1")
   )
-  (symbol (lib_id "74xGxx:74AUC2G125") (at 178.435 107.315 0) (mirror x) (unit 1)
-    (in_bom yes) (on_board yes)
-    (property "Reference" "U9" (id 0) (at 174.625 111.76 0))
-    (property "Value" "74AUC2G125" (id 1) (at 172.72 102.87 0))
-    (property "Footprint" "Package_SO:VSSOP-8_2.4x2.1mm_P0.5mm" (id 2) (at 178.435 107.315 0)
-      (effects (font (size 1.27 1.27)) hide)
-    )
-    (property "Datasheet" "http://www.ti.com/lit/sg/scyt129e/scyt129e.pdf" (id 3) (at 178.435 107.315 0)
-      (effects (font (size 1.27 1.27)) hide)
-    )
-    (pin "4")
-    (pin "8")
-    (pin "1")
-    (pin "2")
-    (pin "6")
-    (pin "3")
-    (pin "5")
-    (pin "7")
-  )
   (symbol (lib_id "power:GND") (at 153.67 207.01 0) (unit 1)
     (in_bom yes) (on_board yes)
@@
       (effects (font (size 1.27 1.27)) (justify right))
     )
-    (property "Value" "470p" (id 1) (at 197.485 116.205 0)
+    (property "Value" "680p" (id 1) (at 197.485 116.205 0)
       (effects (font (size 1.27 1.27)) (justify right))
     )
@@
     (pin "1")
   )
+  (symbol (lib_id "74xGxx:74AUC1G74") (at 149.86 127.635 0) (unit 1)
+    (in_bom yes) (on_board yes) (fields_autoplaced)
+    (property "Reference" "U8" (id 0) (at 151.5301 118.745 0)
+      (effects (font (size 1.27 1.27)) (justify left))
+    )
+    (property "Value" "74LVC2G74DP,125" (id 1) (at 151.5301 121.285 0)
+      (effects (font (size 1.27 1.27)) (justify left))
+    )
+    (property "Footprint" "Package_SO:TSSOP-8_3x3mm_P0.65mm" (id 2) (at 149.86 127.635 0)
+      (effects (font (size 1.27 1.27)) hide)
+    )
+    (property "Datasheet" "http://www.ti.com/lit/sg/scyt129e/scyt129e.pdf" (id 3) (at 149.86 127.635 0)
+      (effects (font (size 1.27 1.27)) hide)
+    )
+    (pin "1")
+    (pin "2")
+    (pin "3")
+    (pin "4")
+    (pin "5")
+    (pin "6")
+    (pin "7")
+    (pin "8")
+  )
   (symbol (lib_id "power:+5V") (at 179.705 110.49 180) (unit 1)
     (in_bom yes) (on_board yes)
@@
   (symbol (lib_id "MCU_Microchip_AVR_Dx:AVR32DB28x-xSO") (at 335.28 85.725 0) (unit 1)
     (in_bom yes) (on_board yes) (fields_autoplaced)
-    (property "Reference" "U12" (id 0) (at 337.2994 109.22 0)
+    (property "Reference" "U13" (id 0) (at 337.2994 109.22 0)
       (effects (font (size 1.27 1.27)) (justify left))
     )
@@
     (pin "2")
   )
-  (symbol (lib_id "74xGxx:74AUC2G125") (at 172.085 125.095 0) (unit 2)
-    (in_bom yes) (on_board yes)
-    (property "Reference" "U9" (id 0) (at 167.64 120.65 0))
-    (property "Value" "74AUC2G125" (id 1) (at 173.355 132.715 0))
-    (property "Footprint" "Package_SO:VSSOP-8_2.4x2.1mm_P0.5mm" (id 2) (at 172.085 125.095 0)
-      (effects (font (size 1.27 1.27)) hide)
-    )
-    (property "Datasheet" "http://www.ti.com/lit/sg/scyt129e/scyt129e.pdf" (id 3) (at 172.085 125.095 0)
-      (effects (font (size 1.27 1.27)) hide)
-    )
-    (pin "4")
-    (pin "8")
-    (pin "1")
-    (pin "2")
-    (pin "6")
-    (pin "3")
-    (pin "5")
-    (pin "7")
-  )
   (symbol (lib_id "Regulator_Linear:L7805") (at 74.93 196.215 0) (unit 1)
     (in_bom yes) (on_board yes) (fields_autoplaced)
@@
     (pin "2")
   )
+  (symbol (lib_id "74xGxx:74AUC1G125") (at 178.435 107.315 0) (mirror x) (unit 1)
+    (in_bom yes) (on_board yes)
+    (property "Reference" "U10" (id 0) (at 177.8 99.06 0))
+    (property "Value" "74LVC1G125SE-7" (id 1) (at 170.815 103.505 0))
+    (property "Footprint" "Package_TO_SOT_SMD:SOT-353_SC-70-5" (id 2) (at 178.435 107.315 0)
+      (effects (font (size 1.27 1.27)) hide)
+    )
+    (property "Datasheet" "http://www.ti.com/lit/sg/scyt129e/scyt129e.pdf" (id 3) (at 178.435 107.315 0)
+      (effects (font (size 1.27 1.27)) hide)
+    )
+    (pin "1")
+    (pin "2")
+    (pin "3")
+    (pin "4")
+    (pin "5")
+  )
   (symbol (lib_id "Transistor_BJT:BC817") (at 95.885 38.735 0) (unit 1)
     (in_bom yes) (on_board yes) (fields_autoplaced)
@@
     (pin "1")
   )
-  (symbol (lib_id "74xGxx:74AUC1G74") (at 149.86 127.635 0) (unit 1)
-    (in_bom yes) (on_board yes) (fields_autoplaced)
-    (property "Reference" "U8" (id 0) (at 151.5301 118.745 0)
-      (effects (font (size 1.27 1.27)) (justify left))
-    )
-    (property "Value" "74AUC1G74" (id 1) (at 151.5301 121.285 0)
-      (effects (font (size 1.27 1.27)) (justify left))
-    )
-    (property "Footprint" "Package_SO:VSSOP-8_2.3x2mm_P0.5mm" (id 2) (at 149.86 127.635 0)
-      (effects (font (size 1.27 1.27)) hide)
-    )
-    (property "Datasheet" "http://www.ti.com/lit/sg/scyt129e/scyt129e.pdf" (id 3) (at 149.86 127.635 0)
-      (effects (font (size 1.27 1.27)) hide)
-    )
-    (pin "1")
-    (pin "2")
-    (pin "3")
-    (pin "4")
-    (pin "5")
-    (pin "6")
-    (pin "7")
-    (pin "8")
-  )
   (symbol (lib_id "74xx:74HC590") (at 226.695 153.035 0) (unit 1)
     (in_bom yes) (on_board yes)
-    (property "Reference" "U10" (id 0) (at 231.775 135.89 0)
+    (property "Reference" "U11" (id 0) (at 231.775 135.89 0)
       (effects (font (size 1.27 1.27)) (justify left))
     )
@@
     (pin "3")
   )
+  (symbol (lib_id "74xGxx:74AUC1G125") (at 172.085 125.095 0) (unit 1)
+    (in_bom yes) (on_board yes)
+    (property "Reference" "U9" (id 0) (at 170.18 128.905 0))
+    (property "Value" "74LVC1G125SE-7" (id 1) (at 171.45 132.715 0))
+    (property "Footprint" "Package_TO_SOT_SMD:SOT-353_SC-70-5" (id 2) (at 172.085 125.095 0)
+      (effects (font (size 1.27 1.27)) hide)
+    )
+    (property "Datasheet" "http://www.ti.com/lit/sg/scyt129e/scyt129e.pdf" (id 3) (at 172.085 125.095 0)
+      (effects (font (size 1.27 1.27)) hide)
+    )
+    (pin "1")
+    (pin "2")
+    (pin "3")
+    (pin "4")
+    (pin "5")
+  )
   (symbol (lib_id "Device:C") (at 117.475 66.675 90) (unit 1)
     (in_bom yes) (on_board yes) (fields_autoplaced)
@@
     (in_bom yes) (on_board yes)
     (property "Reference" "R13" (id 0) (at 189.865 104.775 90))
-    (property "Value" "200R" (id 1) (at 189.865 109.855 90))
+    (property "Value" "150R" (id 1) (at 189.865 109.855 90))
     (property "Footprint" "Resistor_SMD:R_0805_2012Metric_Pad1.20x1.40mm_HandSolder" (id 2) (at 189.865 107.315 0)
       (effects (font (size 1.27 1.27)) hide)
@@
     )
     (path "/3c69436f-a9d4-4db4-9d3c-3fbb89d14cc4"
-      (reference "C19") (unit 1) (value "470p") (footprint "Capacitor_SMD:C_0805_2012Metric_Pad1.18x1.45mm_HandSolder")
+      (reference "C19") (unit 1) (value "680p") (footprint "Capacitor_SMD:C_0805_2012Metric_Pad1.18x1.45mm_HandSolder")
     )
     (path "/7e85b059-ae9e-4bee-a093-a30ddce3b570"
@@
     )
     (path "/e7d29f65-e587-413c-9f79-9a1602df5c7e"
-      (reference "R13") (unit 1) (value "200R") (footprint "Resistor_SMD:R_0805_2012Metric_Pad1.20x1.40mm_HandSolder")
+      (reference "R13") (unit 1) (value "150R") (footprint "Resistor_SMD:R_0805_2012Metric_Pad1.20x1.40mm_HandSolder")
     )
     (path "/424ddaba-b6fc-4f02-af95-a4efad8a4d85"
@@
       (reference "U7") (unit 1) (value "LT1719CS6") (footprint "Package_TO_SOT_SMD_AKL:SOT-23-6")
     )
-    (path "/bdc82b14-9cfe-4a26-bfe3-09c093fb2345"
-      (reference "U8") (unit 1) (value "74AUC1G74") (footprint "Package_SO:VSSOP-8_2.3x2mm_P0.5mm")
-    )
-    (path "/148aad19-f574-4c93-bb15-24d8cefc8f96"
-      (reference "U9") (unit 1) (value "74AUC2G125") (footprint "Package_SO:VSSOP-8_2.4x2.1mm_P0.5mm")
-    )
-    (path "/96957ee7-ece9-4eac-9447-18b1757a6f00"
-      (reference "U9") (unit 2) (value "74AUC2G125") (footprint "Package_SO:VSSOP-8_2.4x2.1mm_P0.5mm")
+    (path "/775d364c-75d4-42f5-a099-d4c41cf1ab12"
+      (reference "U8") (unit 1) (value "74LVC2G74DP,125") (footprint "Package_SO:TSSOP-8_3x3mm_P0.65mm")
+    )
+    (path "/d7757d43-636e-4c4a-8e2d-513d5b6098f4"
+      (reference "U9") (unit 1) (value "74LVC1G125SE-7") (footprint "Package_TO_SOT_SMD:SOT-353_SC-70-5")
+    )
+    (path "/ae30aa14-e01d-4885-92de-b4b661aca297"
+      (reference "U10") (unit 1) (value "74LVC1G125SE-7") (footprint "Package_TO_SOT_SMD:SOT-353_SC-70-5")
     )
     (path "/be55dabe-c026-4082-96e0-5f65c839136b"
-      (reference "U10") (unit 1) (value "74HC590PW,118") (footprint "Package_SO:TSSOP-16_4.4x5mm_P0.65mm")
+      (reference "U11") (unit 1) (value "74HC590PW,118") (footprint "Package_SO:TSSOP-16_4.4x5mm_P0.65mm")
     )
     (path "/10bd52e6-af6a-413e-9c10-f3da44c4133b"
-      (reference "U11") (unit 1) (value "74HCS251") (footprint "Package_SO:SOIC-16_4.55x10.3mm_P1.27mm")
+      (reference "U12") (unit 1) (value "74HCS251") (footprint "Package_SO:SOIC-16_4.55x10.3mm_P1.27mm")
     )
     (path "/8b3913bb-73bc-468d-a4a4-eaf44e1d1389"
-      (reference "U12") (unit 1) (value "AVR32DB28x-xSO") (footprint "Package_SO:SOIC-28W_7.5x17.9mm_P1.27mm")
+      (reference "U13") (unit 1) (value "AVR32DB28x-xSO") (footprint "Package_SO:SOIC-28W_7.5x17.9mm_P1.27mm")
     )
     (path "/933c2574-012e-47d3-94dd-3c3fcd695e78"

Commit message: Updated schematic with correct 5V devices
Parts:
- added C19, C20: 100n, Capacitor_SMD:C_0805_2012Metric_Pad1.18x1.45mm_HandSolder, symbol Device:C
- renumbered C19 to C21, C20 to C22, C21 to C23, C22 to C24, C23 to C25, C24 to C26, C25 to C27, C26 to C28, C27 to C29
Connections:
- net +5V: now also C19.2, C20.2
- net GND: now also C19.1, C20.1
Other:
- note added: "Polystyrene"
- note added: "low parasitic"
- note added: "tantalum"
